File: Eagle files/Universal Bicore (rev A) - 1x3 panelized.brd (EAGLE design)
At the start: 49.8 x 49.8 mm, 66 parts, among them IC1 74HCT240N, IC2 74HCT240N, IC3 74HCT240N

Commit message: Updated panelized PCB
Fixed ground bug in panelized PCB.
Connections:
- removed net GND1: IC2.10, JP12.2, JP20.1, JP21.1, LED3.C, LED4.C
- removed net GND2: IC3.10, JP23.2, JP31.1, JP32.1, LED5.C, LED6.C
- net GND: now also IC2.10, IC3.10, JP12.2, JP20.1, JP21.1, JP23.2, JP31.1, JP32.1, LED3.C, LED4.C, LED5.C, LED6.C
Changed lines of the file:
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@@
 <contactref element="JP10" pad="1"/>
 <contactref element="JP9" pad="1"/>
+<contactref element="IC3" pad="10"/>
+<contactref element="JP23" pad="2"/>
+<contactref element="LED6" pad="C"/>
+<contactref element="LED5" pad="C"/>
+<contactref element="JP32" pad="1"/>
+<contactref element="JP31" pad="1"/>
+<contactref element="IC2" pad="10"/>
+<contactref element="JP12" pad="2"/>
+<contactref element="LED4" pad="C"/>
+<contactref element="LED3" pad="C"/>
+<contactref element="JP21" pad="1"/>
+<contactref element="JP20" pad="1"/>
 </signal>
 <signal name="VCC">
@@
 <wire x1="8.128" y1="41.402" x2="8.382" y2="41.402" width="0.254" layer="1"/>
 </signal>
-<signal name="GND1">
-<contactref element="IC2" pad="10"/>
-<contactref element="JP12" pad="2"/>
-<contactref element="LED4" pad="C"/>
-<contactref element="LED3" pad="C"/>
-<contactref element="JP21" pad="1"/>
-<contactref element="JP20" pad="1"/>
-</signal>
 <signal name="VCC1">
 <contactref element="IC2" pad="20"/>
@@
 <wire x1="41.402" y1="41.402" x2="41.656" y2="41.402" width="0.254" layer="1"/>
 </signal>
-<signal name="GND2">
-<contactref element="IC3" pad="10"/>
-<contactref element="JP23" pad="2"/>
-<contactref element="LED6" pad="C"/>
-<contactref element="LED5" pad="C"/>
-<contactref element="JP32" pad="1"/>
-<contactref element="JP31" pad="1"/>
-</signal>
 <signal name="VCC2">
 <contactref element="IC3" pad="20"/>
@@
 </signal>
 </signals>
-<errors>
-</errors>
 </board>
 </drawing>
